File: MAX31850.sch (KiCad schematic (older format))
At the start: 10 parts, among them U1 MAX31850KATB+

Commit message: Bugfixes in the schematic and started the pcb layout
Connections:
- net at C1.2, C3.1, FB1.1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: now also D1.2 (K); no longer D1.1 (K)
- net at C2.1, C3.2, FB2.1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: now also D1.1 (K); no longer D1.2 (K)
Changed lines of the file:
@@
 $Descr A4 11693 8268
 encoding utf-8
-Sheet 7 9
+Sheet 5 9
 Title "Thermocouple MAX31850"
 Date "2020-10-16"
@@
 AR Path="/5E3E3667/5E3B9C37" Ref="#PWR048"  Part="1"
 AR Path="/5E3E8E80/5E3B9C37" Ref="#PWR056"  Part="1"
-F 0 "#PWR056" H 6000 4450 50  0001 C CNN
+F 0 "#PWR014" H 6000 4450 50  0001 C CNN
 F 1 "VSSA" H 6018 4773 50  0000 C CNN
 F 2 "" H 6000 4600 50  0001 C CNN
@@
 AR Path="/5E3E3667/5E3C8A66" Ref="FB9"  Part="1"
 AR Path="/5E3E8E80/5E3C8A66" Ref="FB11"  Part="1"
-F 0 "FB11" V 3050 4500 50  0000 C CNN
+F 0 "FB9" V 3050 4500 50  0000 C CNN
 F 1 "BLM18PG121SN1D" V 2950 4500 50  0000 C CNN
 F 2 "Inductor_SMD:L_0603_1608Metric" V 2780 4500 50  0001 C CNN
@@
 AR Path="/5E3E3667/5E3D0C8B" Ref="C29"  Part="1"
 AR Path="/5E3E8E80/5E3D0C8B" Ref="C35"  Part="1"
-F 0 "C35" H 8415 3996 50  0000 L CNN
+F 0 "C29" H 8415 3996 50  0000 L CNN
 F 1 "0.1uF" H 8415 3905 50  0000 L CNN
 F 2 "Capacitor_SMD:C_0603_1608Metric" H 8338 3800 50  0001 C CNN
@@
 AR Path="/5E3E3667/5E3DBF02" Ref="C30"  Part="1"
 AR Path="/5E3E8E80/5E3DBF02" Ref="C36"  Part="1"
-F 0 "C36" H 8865 3996 50  0000 L CNN
+F 0 "C30" H 8865 3996 50  0000 L CNN
 F 1 "1uF" H 8865 3905 50  0000 L CNN
 F 2 "Capacitor_SMD:C_0603_1608Metric" H 8788 3800 50  0001 C CNN
@@
 AR Path="/5E3E3667/5E3F83EC" Ref="C28"  Part="1"
 AR Path="/5E3E8E80/5E3F83EC" Ref="C34"  Part="1"
-F 0 "C34" H 7915 3996 50  0000 L CNN
+F 0 "C28" H 7915 3996 50  0000 L CNN
 F 1 "0.01uF" H 7915 3905 50  0000 L CNN
 F 2 "Capacitor_SMD:C_0603_1608Metric" H 7838 3800 50  0001 C CNN
@@
 AR Path="/5E3E3667/5E3C171C" Ref="C27"  Part="1"
 AR Path="/5E3E8E80/5E3C171C" Ref="C33"  Part="1"
-F 0 "C33" H 4265 3996 50  0000 L CNN
+F 0 "C27" H 4265 3996 50  0000 L CNN
 F 1 "0.01uF" H 4265 3905 50  0000 L CNN
 F 2 "Capacitor_SMD:C_0603_1608Metric" H 4188 3800 50  0001 C CNN
@@
 AR Path="/5E3E8E80/5E3B5F5C" Ref="U7"  Part="1"
 AR Path="/5E3B5F5C" Ref="U?"  Part="1"
-F 0 "U7" H 6300 4650 50  0000 C CNN
+F 0 "U6" H 6300 4650 50  0000 C CNN
 F 1 "MAX31850KATB+ " H 6050 4550 50  0000 C CNN
 F 2 "T-962_Upgrade_board:MAX31850" H 6000 3950 50  0001 C CIN
@@
 AR Path="/5E3E3667/5E3C59DE" Ref="FB8"  Part="1"
 AR Path="/5E3E8E80/5E3C59DE" Ref="FB10"  Part="1"
-F 0 "FB10" V 2600 3500 50  0000 C CNN
+F 0 "FB8" V 2600 3500 50  0000 C CNN
 F 1 "BLM18PG121SN1D" V 2700 3500 50  0000 C CNN
 F 2 "Inductor_SMD:L_0603_1608Metric" V 2730 3500 50  0001 C CNN
@@
 AR Path="/5E3E3667/5E3B92B5" Ref="#PWR046"  Part="1"
 AR Path="/5E3E8E80/5E3B92B5" Ref="#PWR054"  Part="1"
-F 0 "#PWR054" H 5050 4100 50  0001 C CNN
+F 0 "#PWR012" H 5050 4100 50  0001 C CNN
 F 1 "VDDA" H 5067 4423 50  0000 C CNN
 F 2 "" H 5050 4250 50  0001 C CNN
@@
 AR Path="/5E3E25D1/5F8E9AAF" Ref="D6"  Part="1"
 AR Path="/5E3E8E80/5F8E9AAF" Ref="D8"  Part="1"
-F 0 "D8" V 3700 3750 50  0000 L CNN
-F 1 "NUP2105L" V 3600 3750 50  0000 L CNN
+F 0 "D7" V 3100 3850 50  0000 L CNN
+F 1 "NUP2105L" V 3000 3750 50  0000 L CNN
 F 2 "Package_TO_SOT_SMD:SOT-23" H 3575 3900 50  0001 L CNN
 F 3 "https://www.onsemi.com/pub/Collateral/NUP2105L-D.PDF" H 3475 4075 50  0001 C CNN
@@
 F 9 "44V Clamp 8A (8/20µs) Ipp Tvs Diode Surface Mount SOT-23-3 (TO-236)" H 3350 3950 50  0001 C CNN "description"
 	1    3350 3950
-	0    1    1    0
+	0    1    -1   0
 $EndComp
 Wire Wire Line
@@
 AR Path="/5E3E25D1/5F8ED8FD" Ref="#PWR035"  Part="1"
 AR Path="/5E3E8E80/5F8ED8FD" Ref="#PWR051"  Part="1"
-F 0 "#PWR051" H 2950 3900 50  0001 C CNN
+F 0 "#PWR09" H 2950 3900 50  0001 C CNN
 F 1 "VSSA" H 2965 4223 50  0000 C CNN
 F 2 "" H 2950 4050 50  0001 C CNN
@@
 AR Path="/5E3E25D1/5F8F1DF2" Ref="#PWR039"  Part="1"
 AR Path="/5E3E8E80/5F8F1DF2" Ref="#PWR055"  Part="1"
-F 0 "#PWR055" H 5600 2850 50  0001 C CNN
+F 0 "#PWR013" H 5600 2850 50  0001 C CNN
 F 1 "VSSA" H 5615 3173 50  0000 C CNN
 F 2 "" H 5600 3000 50  0001 C CNN
@@
 AR Path="/5E3E25D1/5F8FBDE3" Ref="#PWR041"  Part="1"
 AR Path="/5E3E8E80/5F8FBDE3" Ref="#PWR057"  Part="1"
-F 0 "#PWR057" H 8300 3050 50  0001 C CNN
+F 0 "#PWR015" H 8300 3050 50  0001 C CNN
 F 1 "VDDA" H 8315 3373 50  0000 C CNN
 F 2 "" H 8300 3200 50  0001 C CNN
@@
 AR Path="/5E3E25D1/5F8FC217" Ref="#PWR042"  Part="1"
 AR Path="/5E3E8E80/5F8FC217" Ref="#PWR058"  Part="1"
-F 0 "#PWR058" H 8300 4400 50  0001 C CNN
+F 0 "#PWR016" H 8300 4400 50  0001 C CNN
 F 1 "VSSA" H 8315 4723 50  0000 C CNN
 F 2 "" H 8300 4550 50  0001 C CNN
@@
 AR Path="/5E3E25D1/5F9032A0" Ref="C20"  Part="1"
 AR Path="/5E3E8E80/5F9032A0" Ref="C32"  Part="1"
-F 0 "C32" H 3665 4696 50  0000 L CNN
+F 0 "C26" H 3665 4696 50  0000 L CNN
 F 1 "DNP" H 3665 4605 50  0000 L CNN
 F 2 "Capacitor_SMD:C_0603_1608Metric" H 3588 4500 50  0001 C CNN
@@
 AR Path="/5E3E25D1/5F903B97" Ref="#PWR036"  Part="1"
 AR Path="/5E3E8E80/5F903B97" Ref="#PWR052"  Part="1"
-F 0 "#PWR052" H 3550 4700 50  0001 C CNN
+F 0 "#PWR010" H 3550 4700 50  0001 C CNN
 F 1 "VSSA" H 3565 5023 50  0000 C CNN
 F 2 "" H 3550 4850 50  0001 C CNN
@@
 AR Path="/5E3E25D1/5F90502A" Ref="C19"  Part="1"
 AR Path="/5E3E8E80/5F90502A" Ref="C31"  Part="1"
-F 0 "C31" H 3665 3396 50  0000 L CNN
+F 0 "C25" H 3665 3396 50  0000 L CNN
 F 1 "DNP" H 3665 3305 50  0000 L CNN
 F 2 "Capacitor_SMD:C_0603_1608Metric" H 3588 3200 50  0001 C CNN
@@
 AR Path="/5E3E25D1/5F906F5B" Ref="#PWR037"  Part="1"
 AR Path="/5E3E8E80/5F906F5B" Ref="#PWR053"  Part="1"
-F 0 "#PWR053" H 3850 2850 50  0001 C CNN
+F 0 "#PWR011" H 3850 2850 50  0001 C CNN
 F 1 "VSSA" H 3865 3173 50  0000 C CNN
 F 2 "" H 3850 3000 50  0001 C CNN

Commit message: Layout changes
Changed lines of the file:
@@
 $Descr A4 11693 8268
 encoding utf-8
-Sheet 5 9
+Sheet 9 9
 Title "Thermocouple MAX31850"
 Date "2020-10-16"
@@
 AR Path="/5E3E3667/5E3C8A66" Ref="FB9"  Part="1"
 AR Path="/5E3E8E80/5E3C8A66" Ref="FB11"  Part="1"
-F 0 "FB9" V 3050 4500 50  0000 C CNN
+F 0 "FB2" V 3050 4500 50  0000 C CNN
 F 1 "BLM18PG121SN1D" V 2950 4500 50  0000 C CNN
 F 2 "Inductor_SMD:L_0603_1608Metric" V 2780 4500 50  0001 C CNN
@@
 AR Path="/5E3E3667/5E3D0C8B" Ref="C29"  Part="1"
 AR Path="/5E3E8E80/5E3D0C8B" Ref="C35"  Part="1"
-F 0 "C29" H 8415 3996 50  0000 L CNN
+F 0 "C5" H 8415 3996 50  0000 L CNN
 F 1 "0.1uF" H 8415 3905 50  0000 L CNN
 F 2 "Capacitor_SMD:C_0603_1608Metric" H 8338 3800 50  0001 C CNN
@@
 AR Path="/5E3E3667/5E3DBF02" Ref="C30"  Part="1"
 AR Path="/5E3E8E80/5E3DBF02" Ref="C36"  Part="1"
-F 0 "C30" H 8865 3996 50  0000 L CNN
+F 0 "C6" H 8865 3996 50  0000 L CNN
 F 1 "1uF" H 8865 3905 50  0000 L CNN
 F 2 "Capacitor_SMD:C_0603_1608Metric" H 8788 3800 50  0001 C CNN
@@
 AR Path="/5E3E3667/5E3F83EC" Ref="C28"  Part="1"
 AR Path="/5E3E8E80/5E3F83EC" Ref="C34"  Part="1"
-F 0 "C28" H 7915 3996 50  0000 L CNN
+F 0 "C4" H 7915 3996 50  0000 L CNN
 F 1 "0.01uF" H 7915 3905 50  0000 L CNN
 F 2 "Capacitor_SMD:C_0603_1608Metric" H 7838 3800 50  0001 C CNN
@@
 AR Path="/5E3E3667/5E3C171C" Ref="C27"  Part="1"
 AR Path="/5E3E8E80/5E3C171C" Ref="C33"  Part="1"
-F 0 "C27" H 4265 3996 50  0000 L CNN
+F 0 "C3" H 4265 3996 50  0000 L CNN
 F 1 "0.01uF" H 4265 3905 50  0000 L CNN
 F 2 "Capacitor_SMD:C_0603_1608Metric" H 4188 3800 50  0001 C CNN
@@
 AR Path="/5E3E8E80/5E3B5F5C" Ref="U7"  Part="1"
 AR Path="/5E3B5F5C" Ref="U?"  Part="1"
-F 0 "U6" H 6300 4650 50  0000 C CNN
+F 0 "U1" H 6300 4650 50  0000 C CNN
 F 1 "MAX31850KATB+ " H 6050 4550 50  0000 C CNN
 F 2 "T-962_Upgrade_board:MAX31850" H 6000 3950 50  0001 C CIN
@@
 AR Path="/5E3E3667/5E3C59DE" Ref="FB8"  Part="1"
 AR Path="/5E3E8E80/5E3C59DE" Ref="FB10"  Part="1"
-F 0 "FB8" V 2600 3500 50  0000 C CNN
+F 0 "FB1" V 2600 3500 50  0000 C CNN
 F 1 "BLM18PG121SN1D" V 2700 3500 50  0000 C CNN
 F 2 "Inductor_SMD:L_0603_1608Metric" V 2730 3500 50  0001 C CNN
@@
 AR Path="/5E3E25D1/5F8E9AAF" Ref="D6"  Part="1"
 AR Path="/5E3E8E80/5F8E9AAF" Ref="D8"  Part="1"
-F 0 "D7" V 3100 3850 50  0000 L CNN
+F 0 "D1" V 3100 3850 50  0000 L CNN
 F 1 "NUP2105L" V 3000 3750 50  0000 L CNN
 F 2 "Package_TO_SOT_SMD:SOT-23" H 3575 3900 50  0001 L CNN
@@
 AR Path="/5E3E25D1/5F9032A0" Ref="C20"  Part="1"
 AR Path="/5E3E8E80/5F9032A0" Ref="C32"  Part="1"
-F 0 "C26" H 3665 4696 50  0000 L CNN
+F 0 "C2" H 3665 4696 50  0000 L CNN
 F 1 "DNP" H 3665 4605 50  0000 L CNN
 F 2 "Capacitor_SMD:C_0603_1608Metric" H 3588 4500 50  0001 C CNN
@@
 AR Path="/5E3E25D1/5F90502A" Ref="C19"  Part="1"
 AR Path="/5E3E8E80/5F90502A" Ref="C31"  Part="1"
-F 0 "C25" H 3665 3396 50  0000 L CNN
+F 0 "C1" H 3665 3396 50  0000 L CNN
 F 1 "DNP" H 3665 3305 50  0000 L CNN
 F 2 "Capacitor_SMD:C_0603_1608Metric" H 3588 3200 50  0001 C CNN

Commit message: Finished routing
Changed lines of the file:
@@
 $Descr A4 11693 8268
 encoding utf-8
-Sheet 9 9
+Sheet 4 9
 Title "Thermocouple MAX31850"
 Date "2020-10-16"
@@
 AR Path="/5E3E3667/5E3B9C37" Ref="#PWR048"  Part="1"
 AR Path="/5E3E8E80/5E3B9C37" Ref="#PWR056"  Part="1"
-F 0 "#PWR014" H 6000 4450 50  0001 C CNN
+F 0 "#PWR040" H 6000 4450 50  0001 C CNN
 F 1 "VSSA" H 6018 4773 50  0000 C CNN
 F 2 "" H 6000 4600 50  0001 C CNN
@@
 AR Path="/5E3E3667/5E3C8A66" Ref="FB9"  Part="1"
 AR Path="/5E3E8E80/5E3C8A66" Ref="FB11"  Part="1"
-F 0 "FB2" V 3050 4500 50  0000 C CNN
+F 0 "FB7" V 3050 4500 50  0000 C CNN
 F 1 "BLM18PG121SN1D" V 2950 4500 50  0000 C CNN
 F 2 "Inductor_SMD:L_0603_1608Metric" V 2780 4500 50  0001 C CNN
@@
 AR Path="/5E3E3667/5E3D0C8B" Ref="C29"  Part="1"
 AR Path="/5E3E8E80/5E3D0C8B" Ref="C35"  Part="1"
-F 0 "C5" H 8415 3996 50  0000 L CNN
+F 0 "C23" H 8415 3996 50  0000 L CNN
 F 1 "0.1uF" H 8415 3905 50  0000 L CNN
 F 2 "Capacitor_SMD:C_0603_1608Metric" H 8338 3800 50  0001 C CNN
@@
 AR Path="/5E3E3667/5E3DBF02" Ref="C30"  Part="1"
 AR Path="/5E3E8E80/5E3DBF02" Ref="C36"  Part="1"
-F 0 "C6" H 8865 3996 50  0000 L CNN
+F 0 "C24" H 8865 3996 50  0000 L CNN
 F 1 "1uF" H 8865 3905 50  0000 L CNN
 F 2 "Capacitor_SMD:C_0603_1608Metric" H 8788 3800 50  0001 C CNN
@@
 AR Path="/5E3E3667/5E3F83EC" Ref="C28"  Part="1"
 AR Path="/5E3E8E80/5E3F83EC" Ref="C34"  Part="1"
-F 0 "C4" H 7915 3996 50  0000 L CNN
+F 0 "C22" H 7915 3996 50  0000 L CNN
 F 1 "0.01uF" H 7915 3905 50  0000 L CNN
 F 2 "Capacitor_SMD:C_0603_1608Metric" H 7838 3800 50  0001 C CNN
@@
 AR Path="/5E3E3667/5E3C171C" Ref="C27"  Part="1"
 AR Path="/5E3E8E80/5E3C171C" Ref="C33"  Part="1"
-F 0 "C3" H 4265 3996 50  0000 L CNN
+F 0 "C21" H 4265 3996 50  0000 L CNN
 F 1 "0.01uF" H 4265 3905 50  0000 L CNN
 F 2 "Capacitor_SMD:C_0603_1608Metric" H 4188 3800 50  0001 C CNN
@@
 AR Path="/5E3E8E80/5E3B5F5C" Ref="U7"  Part="1"
 AR Path="/5E3B5F5C" Ref="U?"  Part="1"
-F 0 "U1" H 6300 4650 50  0000 C CNN
+F 0 "U5" H 6300 4650 50  0000 C CNN
 F 1 "MAX31850KATB+ " H 6050 4550 50  0000 C CNN
 F 2 "T-962_Upgrade_board:MAX31850" H 6000 3950 50  0001 C CIN
@@
 AR Path="/5E3E3667/5E3C59DE" Ref="FB8"  Part="1"
 AR Path="/5E3E8E80/5E3C59DE" Ref="FB10"  Part="1"
-F 0 "FB1" V 2600 3500 50  0000 C CNN
+F 0 "FB6" V 2600 3500 50  0000 C CNN
 F 1 "BLM18PG121SN1D" V 2700 3500 50  0000 C CNN
 F 2 "Inductor_SMD:L_0603_1608Metric" V 2730 3500 50  0001 C CNN
@@
 AR Path="/5E3E3667/5E3B92B5" Ref="#PWR046"  Part="1"
 AR Path="/5E3E8E80/5E3B92B5" Ref="#PWR054"  Part="1"
-F 0 "#PWR012" H 5050 4100 50  0001 C CNN
+F 0 "#PWR038" H 5050 4100 50  0001 C CNN
 F 1 "VDDA" H 5067 4423 50  0000 C CNN
 F 2 "" H 5050 4250 50  0001 C CNN
@@
 AR Path="/5E3E25D1/5F8E9AAF" Ref="D6"  Part="1"
 AR Path="/5E3E8E80/5F8E9AAF" Ref="D8"  Part="1"
-F 0 "D1" V 3100 3850 50  0000 L CNN
+F 0 "D6" V 3100 3850 50  0000 L CNN
 F 1 "NUP2105L" V 3000 3750 50  0000 L CNN
 F 2 "Package_TO_SOT_SMD:SOT-23" H 3575 3900 50  0001 L CNN
@@
 AR Path="/5E3E25D1/5F8ED8FD" Ref="#PWR035"  Part="1"
 AR Path="/5E3E8E80/5F8ED8FD" Ref="#PWR051"  Part="1"
-F 0 "#PWR09" H 2950 3900 50  0001 C CNN
+F 0 "#PWR035" H 2950 3900 50  0001 C CNN
 F 1 "VSSA" H 2965 4223 50  0000 C CNN
 F 2 "" H 2950 4050 50  0001 C CNN
@@
 AR Path="/5E3E25D1/5F8F1DF2" Ref="#PWR039"  Part="1"
 AR Path="/5E3E8E80/5F8F1DF2" Ref="#PWR055"  Part="1"
-F 0 "#PWR013" H 5600 2850 50  0001 C CNN
+F 0 "#PWR039" H 5600 2850 50  0001 C CNN
 F 1 "VSSA" H 5615 3173 50  0000 C CNN
 F 2 "" H 5600 3000 50  0001 C CNN
@@
 AR Path="/5E3E25D1/5F8FBDE3" Ref="#PWR041"  Part="1"
 AR Path="/5E3E8E80/5F8FBDE3" Ref="#PWR057"  Part="1"
-F 0 "#PWR015" H 8300 3050 50  0001 C CNN
+F 0 "#PWR041" H 8300 3050 50  0001 C CNN
 F 1 "VDDA" H 8315 3373 50  0000 C CNN
 F 2 "" H 8300 3200 50  0001 C CNN
@@
 AR Path="/5E3E25D1/5F8FC217" Ref="#PWR042"  Part="1"
 AR Path="/5E3E8E80/5F8FC217" Ref="#PWR058"  Part="1"
-F 0 "#PWR016" H 8300 4400 50  0001 C CNN
+F 0 "#PWR042" H 8300 4400 50  0001 C CNN
 F 1 "VSSA" H 8315 4723 50  0000 C CNN
 F 2 "" H 8300 4550 50  0001 C CNN
@@
 AR Path="/5E3E25D1/5F9032A0" Ref="C20"  Part="1"
 AR Path="/5E3E8E80/5F9032A0" Ref="C32"  Part="1"
-F 0 "C2" H 3665 4696 50  0000 L CNN
+F 0 "C20" H 3665 4696 50  0000 L CNN
 F 1 "DNP" H 3665 4605 50  0000 L CNN
 F 2 "Capacitor_SMD:C_0603_1608Metric" H 3588 4500 50  0001 C CNN
@@
 AR Path="/5E3E25D1/5F903B97" Ref="#PWR036"  Part="1"
 AR Path="/5E3E8E80/5F903B97" Ref="#PWR052"  Part="1"
-F 0 "#PWR010" H 3550 4700 50  0001 C CNN
+F 0 "#PWR036" H 3550 4700 50  0001 C CNN
 F 1 "VSSA" H 3565 5023 50  0000 C CNN
 F 2 "" H 3550 4850 50  0001 C CNN
@@
 AR Path="/5E3E25D1/5F90502A" Ref="C19"  Part="1"
 AR Path="/5E3E8E80/5F90502A" Ref="C31"  Part="1"
-F 0 "C1" H 3665 3396 50  0000 L CNN
+F 0 "C19" H 3665 3396 50  0000 L CNN
 F 1 "DNP" H 3665 3305 50  0000 L CNN
 F 2 "Capacitor_SMD:C_0603_1608Metric" H 3588 3200 50  0001 C CNN
@@
 AR Path="/5E3E25D1/5F906F5B" Ref="#PWR037"  Part="1"
 AR Path="/5E3E8E80/5F906F5B" Ref="#PWR053"  Part="1"
-F 0 "#PWR011" H 3850 2850 50  0001 C CNN
+F 0 "#PWR037" H 3850 2850 50  0001 C CNN
 F 1 "VSSA" H 3865 3173 50  0000 C CNN
 F 2 "" H 3850 3000 50  0001 C CNN

Commit message: small bugfixes. Added parts to bom
Changed lines of the file:
@@
 $Descr A4 11693 8268
 encoding utf-8
-Sheet 4 9
+Sheet 9 9
 Title "Thermocouple MAX31850"
 Date "2020-10-16"
@@
 AR Path="/5E3E3667/5E3B9C37" Ref="#PWR048"  Part="1"
 AR Path="/5E3E8E80/5E3B9C37" Ref="#PWR056"  Part="1"
-F 0 "#PWR040" H 6000 4450 50  0001 C CNN
+F 0 "#PWR014" H 6000 4450 50  0001 C CNN
 F 1 "VSSA" H 6018 4773 50  0000 C CNN
 F 2 "" H 6000 4600 50  0001 C CNN
@@
 AR Path="/5E3E3667/5E3C8A66" Ref="FB9"  Part="1"
 AR Path="/5E3E8E80/5E3C8A66" Ref="FB11"  Part="1"
-F 0 "FB7" V 3050 4500 50  0000 C CNN
+F 0 "FB2" V 3050 4500 50  0000 C CNN
 F 1 "BLM18PG121SN1D" V 2950 4500 50  0000 C CNN
 F 2 "Inductor_SMD:L_0603_1608Metric" V 2780 4500 50  0001 C CNN
@@
 AR Path="/5E3E3667/5E3D0C8B" Ref="C29"  Part="1"
 AR Path="/5E3E8E80/5E3D0C8B" Ref="C35"  Part="1"
-F 0 "C23" H 8415 3996 50  0000 L CNN
+F 0 "C5" H 8415 3996 50  0000 L CNN
 F 1 "0.1uF" H 8415 3905 50  0000 L CNN
 F 2 "Capacitor_SMD:C_0603_1608Metric" H 8338 3800 50  0001 C CNN
@@
 F 10 "1276-CL10B104KB8NNNLCT-ND" H 8300 3950 50  0001 C CNN "SPN"
 F 11 "0.1µF ±10% 50V Ceramic Capacitor X7R 0603 (1608 Metric)" H 8300 3950 50  0001 C CNN "description"
+F 12 "" H 8300 3950 50  0001 C CNN "Assembly"
 	1    8300 3950
 	1    0    0    -1
@@
 AR Path="/5E3E3667/5E3DBF02" Ref="C30"  Part="1"
 AR Path="/5E3E8E80/5E3DBF02" Ref="C36"  Part="1"
-F 0 "C24" H 8865 3996 50  0000 L CNN
+F 0 "C6" H 8865 3996 50  0000 L CNN
 F 1 "1uF" H 8865 3905 50  0000 L CNN
 F 2 "Capacitor_SMD:C_0603_1608Metric" H 8788 3800 50  0001 C CNN
@@
 AR Path="/5E3E3667/5E3F83EC" Ref="C28"  Part="1"
 AR Path="/5E3E8E80/5E3F83EC" Ref="C34"  Part="1"
-F 0 "C22" H 7915 3996 50  0000 L CNN
+F 0 "C4" H 7915 3996 50  0000 L CNN
 F 1 "0.01uF" H 7915 3905 50  0000 L CNN
 F 2 "Capacitor_SMD:C_0603_1608Metric" H 7838 3800 50  0001 C CNN
@@
 AR Path="/5E3E3667/5E3C171C" Ref="C27"  Part="1"
 AR Path="/5E3E8E80/5E3C171C" Ref="C33"  Part="1"
-F 0 "C21" H 4265 3996 50  0000 L CNN
+F 0 "C3" H 4265 3996 50  0000 L CNN
 F 1 "0.01uF" H 4265 3905 50  0000 L CNN
 F 2 "Capacitor_SMD:C_0603_1608Metric" H 4188 3800 50  0001 C CNN
@@
 AR Path="/5E3E8E80/5E3B5F5C" Ref="U7"  Part="1"
 AR Path="/5E3B5F5C" Ref="U?"  Part="1"
-F 0 "U5" H 6300 4650 50  0000 C CNN
+F 0 "U1" H 6300 4650 50  0000 C CNN
 F 1 "MAX31850KATB+ " H 6050 4550 50  0000 C CNN
 F 2 "T-962_Upgrade_board:MAX31850" H 6000 3950 50  0001 C CIN
@@
 F 10 "700-MAX31850KATB+" H 6000 3950 50  0001 C CNN "SPN"
 F 11 "Sensor Interface 1-WIRE THRMOCPLE TO DIG CONV K TYPE " H 6000 3950 50  0001 C CNN "description"
+F 12 "" H 6000 3950 50  0001 C CNN "Assembly"
 	1    6000 3950
 	1    0    0    -1
@@
 AR Path="/5E3E3667/5E3C59DE" Ref="FB8"  Part="1"
 AR Path="/5E3E8E80/5E3C59DE" Ref="FB10"  Part="1"
-F 0 "FB6" V 2600 3500 50  0000 C CNN
+F 0 "FB1" V 2600 3500 50  0000 C CNN
 F 1 "BLM18PG121SN1D" V 2700 3500 50  0000 C CNN
 F 2 "Inductor_SMD:L_0603_1608Metric" V 2730 3500 50  0001 C CNN
@@
 AR Path="/5E3E3667/5E3B92B5" Ref="#PWR046"  Part="1"
 AR Path="/5E3E8E80/5E3B92B5" Ref="#PWR054"  Part="1"
-F 0 "#PWR038" H 5050 4100 50  0001 C CNN
+F 0 "#PWR012" H 5050 4100 50  0001 C CNN
 F 1 "VDDA" H 5067 4423 50  0000 C CNN
 F 2 "" H 5050 4250 50  0001 C CNN
@@
 AR Path="/5E3E25D1/5F8E9AAF" Ref="D6"  Part="1"
 AR Path="/5E3E8E80/5F8E9AAF" Ref="D8"  Part="1"
-F 0 "D6" V 3100 3850 50  0000 L CNN
+F 0 "D1" V 3100 3850 50  0000 L CNN
 F 1 "NUP2105L" V 3000 3750 50  0000 L CNN
 F 2 "Package_TO_SOT_SMD:SOT-23" H 3575 3900 50  0001 L CNN
@@
 AR Path="/5E3E25D1/5F8ED8FD" Ref="#PWR035"  Part="1"
 AR Path="/5E3E8E80/5F8ED8FD" Ref="#PWR051"  Part="1"
-F 0 "#PWR035" H 2950 3900 50  0001 C CNN
+F 0 "#PWR09" H 2950 3900 50  0001 C CNN
 F 1 "VSSA" H 2965 4223 50  0000 C CNN
 F 2 "" H 2950 4050 50  0001 C CNN
@@
 AR Path="/5E3E25D1/5F8F1DF2" Ref="#PWR039"  Part="1"
 AR Path="/5E3E8E80/5F8F1DF2" Ref="#PWR055"  Part="1"
-F 0 "#PWR039" H 5600 2850 50  0001 C CNN
+F 0 "#PWR013" H 5600 2850 50  0001 C CNN
 F 1 "VSSA" H 5615 3173 50  0000 C CNN
 F 2 "" H 5600 3000 50  0001 C CNN
@@
 AR Path="/5E3E25D1/5F8FBDE3" Ref="#PWR041"  Part="1"
 AR Path="/5E3E8E80/5F8FBDE3" Ref="#PWR057"  Part="1"
-F 0 "#PWR041" H 8300 3050 50  0001 C CNN
+F 0 "#PWR015" H 8300 3050 50  0001 C CNN
 F 1 "VDDA" H 8315 3373 50  0000 C CNN
 F 2 "" H 8300 3200 50  0001 C CNN
@@
 AR Path="/5E3E25D1/5F8FC217" Ref="#PWR042"  Part="1"
 AR Path="/5E3E8E80/5F8FC217" Ref="#PWR058"  Part="1"
-F 0 "#PWR042" H 8300 4400 50  0001 C CNN
+F 0 "#PWR016" H 8300 4400 50  0001 C CNN
 F 1 "VSSA" H 8315 4723 50  0000 C CNN
 F 2 "" H 8300 4550 50  0001 C CNN
@@
 AR Path="/5E3E25D1/5F9032A0" Ref="C20"  Part="1"
 AR Path="/5E3E8E80/5F9032A0" Ref="C32"  Part="1"
-F 0 "C20" H 3665 4696 50  0000 L CNN
+F 0 "C2" H 3665 4696 50  0000 L CNN
 F 1 "DNP" H 3665 4605 50  0000 L CNN
 F 2 "Capacitor_SMD:C_0603_1608Metric" H 3588 4500 50  0001 C CNN
@@
 AR Path="/5E3E25D1/5F903B97" Ref="#PWR036"  Part="1"
 AR Path="/5E3E8E80/5F903B97" Ref="#PWR052"  Part="1"
-F 0 "#PWR036" H 3550 4700 50  0001 C CNN
+F 0 "#PWR010" H 3550 4700 50  0001 C CNN
 F 1 "VSSA" H 3565 5023 50  0000 C CNN
 F 2 "" H 3550 4850 50  0001 C CNN
@@
 AR Path="/5E3E25D1/5F90502A" Ref="C19"  Part="1"
 AR Path="/5E3E8E80/5F90502A" Ref="C31"  Part="1"
-F 0 "C19" H 3665 3396 50  0000 L CNN
+F 0 "C1" H 3665 3396 50  0000 L CNN
 F 1 "DNP" H 3665 3305 50  0000 L CNN
 F 2 "Capacitor_SMD:C_0603_1608Metric" H 3588 3200 50  0001 C CNN
@@
 AR Path="/5E3E25D1/5F906F5B" Ref="#PWR037"  Part="1"
 AR Path="/5E3E8E80/5F906F5B" Ref="#PWR053"  Part="1"
-F 0 "#PWR037" H 3850 2850 50  0001 C CNN
+F 0 "#PWR011" H 3850 2850 50  0001 C CNN
 F 1 "VSSA" H 3865 3173 50  0000 C CNN
 F 2 "" H 3850 3000 50  0001 C CNN
