File: T962upgrade.sch (KiCad schematic (older format))
At the start: 8 parts, among them J1 Thermalcouple Screw Terminal, J2 2,54mm Pin Header, J3 GPIO Screw Terminal

Commit message: Bugfixes in the schematic and started the pcb layout
Connections:
- net AD0: now also J3.2 (Pin_2); no longer J3.1 (Pin_1)
- net SW_IO: now also J3.1 (Pin_1); no longer J3.2 (Pin_2)
- net Thermocouple 1/T+: now also J1.2 (Pin_2); no longer J1.1 (Pin_1)
- net Thermocouple 1/T-: now also J1.1 (Pin_1); no longer J1.2 (Pin_2)
- net Thermocouple 2/T+: now also J1.4 (Pin_4); no longer J1.3 (Pin_3)
- net Thermocouple 2/T-: now also J1.3 (Pin_3); no longer J1.4 (Pin_4)
- net Thermocouple 3/T+: now also J1.6 (Pin_6); no longer J1.5 (Pin_5)
- net Thermocouple 3/T-: now also J1.5 (Pin_5); no longer J1.6 (Pin_6)
- net Thermocouple 4/T+: now also J1.8 (Pin_8); no longer J1.7 (Pin_7)
- net Thermocouple 4/T-: now also J1.7 (Pin_7); no longer J1.8 (Pin_8)
Changed lines of the file:
@@
 $EndDescr
-$Sheet
-S 3350 1400 1000 1000
-U 5E3B5CB9
-F0 "Thermocouple 1" 50
-F1 "MAX31850.sch" 50
-F2 "SW_IO" B R 4350 1900 50
-F3 "AD0" I L 3350 1500 50
-F4 "AD1" I L 3350 1600 50
-F5 "T-" U L 3350 2250 50
-F6 "T+" U L 3350 2100 50
-$EndSheet
 $Sheet
 S 5000 5600 1000 1000
@@
 F3 "AD0" I L 3350 2900 50
 F4 "AD1" I L 3350 3000 50
-F5 "T-" U L 3350 3650 50
-F6 "T+" U L 3350 3500 50
+F5 "T-" U L 3350 3500 50
+F6 "T+" U L 3350 3650 50
 $EndSheet
 $Sheet
@@
 F3 "AD0" I L 3350 4300 50
 F4 "AD1" I L 3350 4400 50
-F5 "T-" U L 3350 5050 50
-F6 "T+" U L 3350 4900 50
+F5 "T-" U L 3350 4900 50
+F6 "T+" U L 3350 5050 50
 $EndSheet
 $Sheet
@@
 F3 "AD0" I L 3350 5700 50
 F4 "AD1" I L 3350 5800 50
-F5 "T-" U L 3350 6450 50
-F6 "T+" U L 3350 6300 50
+F5 "T-" U L 3350 6300 50
+F6 "T+" U L 3350 6450 50
 $EndSheet
 $Comp
@@
 L Connector:Screw_Terminal_01x02 J?
 U 1 1 5F91E791
-P 7400 2200
+P 7400 2100
 AR Path="/5E3B5CB9/5F91E791" Ref="J?"  Part="1"
 AR Path="/5E3E25D1/5F91E791" Ref="J?"  Part="1"
@@
 AR Path="/5E4C66F1/5F91E791" Ref="J?"  Part="1"
 AR Path="/5F91E791" Ref="J3"  Part="1"
-F 0 "J3" H 7100 2400 50  0000 C CNN
-F 1 "GPIO Screw Terminal" H 7450 2300 50  0000 C CNN
-F 2 "T-962_Upgrade_board:PHOENIX_1985823" H 7400 2200 50  0001 C CNN
-F 3 "https://media.digikey.com/pdf/Data%20Sheets/Phoenix%20Contact%20PDFs/Multi-Postion%20PCTerminal%20Blocks.pdf" H 7400 2200 50  0001 C CNN
-F 4 "WJ15EDGRC-3.81-2P | WJ15EDGK-3.81-2P" H 7400 2200 50  0001 C CNN "manf#"
-F 5 "C8387 | C8466" H 7400 2200 50  0001 C CNN "lcsc#"
-F 6 "https://www.digikey.de/product-detail/en/phoenix-contact/1985823/277-11025-ND/2511042?cur=EUR&lang=en" H 7400 2200 50  0001 C CNN "Link"
-F 7 "1985823" H 7400 2200 50  0001 C CNN "MPN"
-F 8 "Phoenix Contact" H 7400 2200 50  0001 C CNN "Manufacturer"
-F 9 "277-11025-ND" H 7400 2200 50  0001 C CNN "SPN"
-F 10 "2 Position Wire to Board Terminal Block Horizontal with Board 0.150\" (3.81mm) Through Hole" H 7400 2200 50  0001 C CNN "description"
-	1    7400 2200
-	1    0    0    1
+F 0 "J3" H 7400 1900 50  0000 C CNN
+F 1 "GPIO Screw Terminal" H 7450 1800 50  0000 C CNN
+F 2 "T-962_Upgrade_board:PHOENIX_1985823" H 7400 2100 50  0001 C CNN
+F 3 "https://media.digikey.com/pdf/Data%20Sheets/Phoenix%20Contact%20PDFs/Multi-Postion%20PCTerminal%20Blocks.pdf" H 7400 2100 50  0001 C CNN
+F 4 "WJ15EDGRC-3.81-2P | WJ15EDGK-3.81-2P" H 7400 2100 50  0001 C CNN "manf#"
+F 5 "C8387 | C8466" H 7400 2100 50  0001 C CNN "lcsc#"
+F 6 "https://www.digikey.de/product-detail/en/phoenix-contact/1985823/277-11025-ND/2511042?cur=EUR&lang=en" H 7400 2100 50  0001 C CNN "Link"
+F 7 "1985823" H 7400 2100 50  0001 C CNN "MPN"
+F 8 "Phoenix Contact" H 7400 2100 50  0001 C CNN "Manufacturer"
+F 9 "277-11025-ND" H 7400 2100 50  0001 C CNN "SPN"
+F 10 "2 Position Wire to Board Terminal Block Horizontal with Board 0.150\" (3.81mm) Through Hole" H 7400 2100 50  0001 C CNN "description"
+	1    7400 2100
+	1    0    0    -1
 $EndComp
 $Comp
@@
 	4650 1900 4650 1550
 Connection ~ 4650 1900
+$Sheet
+S 3350 1400 1000 1000
+U 5E3B5CB9
+F0 "Thermocouple 1" 50
+F1 "MAX31850.sch" 50
+F2 "SW_IO" B R 4350 1900 50
+F3 "AD0" I L 3350 1500 50
+F4 "AD1" I L 3350 1600 50
+F5 "T-" U L 3350 2100 50
+F6 "T+" U L 3350 2250 50
+$EndSheet
 $EndSCHEMATC

Commit message: Layout changes
Parts:
- H1, H2, H3, H4: Assembly (none) -> DNP
Changed lines of the file:
@@
 F 2 "MountingHole:MountingHole_3.2mm_M3_Pad" H 9000 5350 50  0001 C CNN
 F 3 "~" H 9000 5350 50  0001 C CNN
+F 4 "DNP" H 9000 5350 50  0001 C CNN "Assembly"
 	1    9000 5350
 	1    0    0    -1
@@
 F 2 "MountingHole:MountingHole_3.2mm_M3_Pad" H 9850 5350 50  0001 C CNN
 F 3 "~" H 9850 5350 50  0001 C CNN
+F 4 "DNP" H 9850 5350 50  0001 C CNN "Assembly"
 	1    9850 5350
 	1    0    0    -1
@@
 F 2 "MountingHole:MountingHole_3.2mm_M3_Pad" H 9000 5700 50  0001 C CNN
 F 3 "~" H 9000 5700 50  0001 C CNN
+F 4 "DNP" H 9000 5700 50  0001 C CNN "Assembly"
 	1    9000 5700
 	1    0    0    -1
@@
 F 2 "MountingHole:MountingHole_3.2mm_M3_Pad" H 9850 5700 50  0001 C CNN
 F 3 "~" H 9850 5700 50  0001 C CNN
+F 4 "DNP" H 9850 5700 50  0001 C CNN "Assembly"
 	1    9850 5700
 	1    0    0    -1

Commit message: small bugfixes. Added parts to bom
Parts:
- J1: Package (none) -> THT
- J3: Package (none) -> THT; lcsc# C8387 | C8466 -> (none); manf# WJ15EDGRC-3.81-2P | WJ15EDGK-3.81-2P -> (none)
- R1: Link (none) -> https://www.reichelt.de/de/en/smd-resistor-0603-4-7-kohm-63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; MPN (none) -> RND1550603SAF4701T5E; Manufacturer (none) -> RND COMPONENTS; Package (none) -> 0603 (1608 Metric); SPN (none) -> RND 0603 1 4,7K; description (none) -> Thick film SMD resistor 0603; lcsc# C23162 -> (none); manf# 0603WAF4701T5E -> (none)
Changed lines of the file:
@@
 F 1 "4k7" H 4580 1355 50  0000 R CNN
 F 2 "Resistor_SMD:R_0603_1608Metric" V 4580 1400 50  0001 C CNN
-F 3 "~" H 4650 1400 50  0001 C CNN
-F 4 "C23162" H 4650 1400 50  0001 C CNN "lcsc#"
-F 5 "0603WAF4701T5E" H 4650 1400 50  0001 C CNN "manf#"
+F 3 "https://cdn-reichelt.de/documents/datenblatt/B300/RND_SMD_0603_RESISTOR_2017.pdf" H 4650 1400 50  0001 C CNN
+F 4 "" H 4650 1400 50  0001 C CNN "lcsc#"
+F 5 "" H 4650 1400 50  0001 C CNN "manf#"
+F 6 "https://www.reichelt.de/de/en/smd-resistor-0603-4-7-kohm-63-mw-1--rnd-0603-1-4-7k-p183069.html?r=1" H 4650 1400 50  0001 C CNN "Link"
+F 7 "RND1550603SAF4701T5E" H 4650 1400 50  0001 C CNN "MPN"
+F 8 "RND COMPONENTS" H 4650 1400 50  0001 C CNN "Manufacturer"
+F 9 "0603 (1608 Metric)" H 4650 1400 50  0001 C CNN "Package"
+F 10 "RND 0603 1 4,7K" H 4650 1400 50  0001 C CNN "SPN"
+F 11 "Thick film SMD resistor 0603" H 4650 1400 50  0001 C CNN "description"
+F 12 "" H 4650 1400 50  0001 C CNN "Assembly"
 	1    4650 1400
 	-1   0    0    -1
@@
 F 7 "https://www.digikey.de/product-detail/en/w%C3%BCrth-elektronik/691243310008/732-691243310008-ND/11477812" H 1800 3950 50  0001 C CNN "Link"
 F 8 "8 Position Wire to Board Terminal Block Horizontal with Board 0.150\" (3.81mm) Through Hole" H 1800 3950 50  0001 C CNN "description"
+F 9 "THT" H 1800 3950 50  0001 C CNN "Package"
+F 10 "" H 1800 3950 50  0001 C CNN "Assembly"
 	1    1800 3950
 	-1   0    0    -1
@@
 F 2 "T-962_Upgrade_board:PHOENIX_1985823" H 7400 2100 50  0001 C CNN
 F 3 "https://media.digikey.com/pdf/Data%20Sheets/Phoenix%20Contact%20PDFs/Multi-Postion%20PCTerminal%20Blocks.pdf" H 7400 2100 50  0001 C CNN
-F 4 "WJ15EDGRC-3.81-2P | WJ15EDGK-3.81-2P" H 7400 2100 50  0001 C CNN "manf#"
-F 5 "C8387 | C8466" H 7400 2100 50  0001 C CNN "lcsc#"
+F 4 "" H 7400 2100 50  0001 C CNN "manf#"
+F 5 "" H 7400 2100 50  0001 C CNN "lcsc#"
 F 6 "https://www.digikey.de/product-detail/en/phoenix-contact/1985823/277-11025-ND/2511042?cur=EUR&lang=en" H 7400 2100 50  0001 C CNN "Link"
 F 7 "1985823" H 7400 2100 50  0001 C CNN "MPN"
@@
 F 9 "277-11025-ND" H 7400 2100 50  0001 C CNN "SPN"
 F 10 "2 Position Wire to Board Terminal Block Horizontal with Board 0.150\" (3.81mm) Through Hole" H 7400 2100 50  0001 C CNN "description"
+F 11 "THT" H 7400 2100 50  0001 C CNN "Package"
 	1    7400 2100
 	1    0    0    -1
