File: T962upgrade.kicad_pcb (KiCad board)
At the start: 2 copper layers, 82.9 x 51 mm, 91 parts, among them J1 Thermalcouple Screw Terminal, J2 2,54mm Pin Header, J3 GPIO Screw Terminal, J4 USB_B_Micro, J5 Fan In, J6 Fan Out, Q1 2N7002, SW1 Boot, SW2 Boot, U1 MAX31850KATB+, U2 CH340C, U3 LM1117-3.3, U4 LM1117-3.3, U5 MAX31850KATB+, U6 MAX31850KATB+, U7 MAX31850KATB+, U8 DS18S20

Commit message: Bugfixes in the schematic and started the pcb layout
Parts:
- moved R5 106.8 mm to (124.2, 83.8)
- moved D5 99.3 mm to (127.3, 83.8), turned to 180 degrees
- moved FB3 76.9 mm to (182.8, 108.1), turned to 0 degrees
- moved R4 76.6 mm to (155.9, 126.3), turned to 180 degrees
- moved C7 73.2 mm to (180.1, 105.8), turned to 270 degrees
- moved D4 71.2 mm to (152.9, 126.3)
- moved U4 64.4 mm to (144.3, 110.0), turned to 270 degrees
- moved R7 63.5 mm to (173.5, 85.3), turned to 90 degrees
- moved R6 61.9 mm to (170.9, 85.3), turned to 90 degrees
- moved C19 60.9 mm to (119.8, 96.0), turned to 180 degrees
- moved R8 60.5 mm to (168.4, 85.3), turned to 90 degrees
- moved R9 59.2 mm to (165.9, 85.3), turned to 90 degrees
- moved C20 58.2 mm to (119.8, 101.1), turned to 0 degrees
- moved C31 57.3 mm to (119.8, 113.5), turned to 180 degrees
- moved R2 56.5 mm to (178.1, 93.0)
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Connections:
- D1 pad 1: Net-(C1-Pad2) -> Net-(C2-Pad1)
- D1 pad 2: Net-(C2-Pad1) -> Net-(C1-Pad2)
- D5 pad 1: VSS -> VSSA
- D6 pad 1: Net-(C19-Pad2) -> Net-(C20-Pad1)
- D6 pad 2: Net-(C20-Pad1) -> Net-(C19-Pad2)
- D7 pad 1: Net-(C25-Pad2) -> Net-(C26-Pad1)
- D7 pad 2: Net-(C26-Pad1) -> Net-(C25-Pad2)
- D8 pad 1: Net-(C31-Pad2) -> Net-(C32-Pad1)
- D8 pad 2: Net-(C32-Pad1) -> Net-(C31-Pad2)
- J1 pad 1: /Thermocouple 1/T+ -> /Thermocouple 1/T-
- J1 pad 2: /Thermocouple 1/T- -> /Thermocouple 1/T+
- J1 pad 3: /Thermocouple 2/T+ -> /Thermocouple 2/T-
- J1 pad 4: /Thermocouple 2/T- -> /Thermocouple 2/T+
- J1 pad 5: /Thermocouple 3/T+ -> /Thermocouple 3/T-
- J1 pad 6: /Thermocouple 3/T- -> /Thermocouple 3/T+
- J1 pad 7: /Thermocouple 4/T+ -> /Thermocouple 4/T-
- J1 pad 8: /Thermocouple 4/T- -> /Thermocouple 4/T+
- J3 pad 1: /AD0 -> /SW_IO
- J3 pad 2: /SW_IO -> /AD0
Routing:
- net Net-(D10-Pad2): track 0.76 -> 0.00 mm
- net /AD0: track 0.74 -> 0.00 mm
- net VSSA: track 6.68 -> 5.98 mm
- net Net-(C26-Pad1): track 0.62 -> 0.00 mm
- net Net-(C32-Pad1): track 0.62 -> 0.00 mm
- net Net-(C20-Pad1): track 0.62 -> 0.00 mm
- net Net-(C2-Pad1): track 0.62 -> 0.00 mm
Other:
- board text added: "SW_IO"
- board text removed: "+"
- board text removed: "-"
- board text removed: "SW IO"

Commit message: Layout changes
Parts:
- moved J2 47.8 mm to (153.7, 126.5)
- moved R9 38.4 mm to (153.7, 121.7), turned to 270 degrees
- moved R6 38.4 mm to (158.8, 121.7), turned to 270 degrees
- moved R8 38.4 mm to (156.3, 121.7), turned to 270 degrees
- moved R7 38.4 mm to (161.4, 121.7), turned to 270 degrees
- moved D3 37.0 mm to (157.0, 116.5), turned to 90 degrees
- moved SW1 35.5 mm to (137.2, 125.2)
- moved R3 33.7 mm to (157.0, 113.5), turned to 270 degrees
- moved D2 30.0 mm to (163.3, 116.5), turned to 90 degrees
- moved R2 25.2 mm to (163.3, 113.5), turned to 270 degrees
- moved SW2 16.5 mm to (147.3, 125.2)
- moved C12 14.0 mm to (150.9, 100.0)
- moved C13 14.0 mm to (152.7, 100.2)
- moved C11 13.9 mm to (143.3, 94.4)
- moved C10 13.9 mm to (143.2, 92.7)
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Routing:
- net VDD: track 0.80 -> 0.21 mm
Other:
- board size 82.9 x 51 mm -> 70.5 x 51 mm
- board text added: "+"
- board text added: "-"
- board text added: "PWR_ANALOG"

Commit message: Finished routing
Parts:
- moved C14 10.8 mm to (150.7, 107.9), turned to 270 degrees
- moved C15 8.17 mm to (148.9, 107.7), turned to 270 degrees
- moved D4 3.92 mm to (156.2, 116.1)
- moved R4 3.92 mm to (156.2, 113.0)
- moved R3 3.22 mm to (160.2, 113.0)
- moved D3 3.22 mm to (160.2, 116.2)
- moved D10 2.91 mm to (163.3, 87.4)
- moved D9 2.91 mm to (147.4, 89.4)
- moved J5 2.91 mm to (149.2, 81.7)
- moved J6 2.91 mm to (159.4, 81.7)
- moved Q1 2.91 mm to (158.0, 87.4)
- moved C39 2.91 mm to (150.4, 86.6)
- moved R10 2.91 mm to (154.7, 86.3)
- moved C38 1.72 mm to (132.1, 96.3), turned to 90 degrees
- moved U4 1.38 mm to (143.3, 109.1), turned to 180 degrees
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Routing:
- net VDDA: track 0.00 -> 87.2 mm
- net VDD: track 0.21 -> 72.7 mm
- net /SW_IO: track 0.00 -> 61.5 mm, vias 0 -> 4
- net Net-(C39-Pad1): track 0.00 -> 30.5 mm
- net /AD0: track 0.00 -> 25.4 mm
- net Net-(R8-Pad1): track 0.00 -> 24.6 mm
- net +VDC: track 0.00 -> 24.3 mm, vias 0 -> 2
- net Net-(R6-Pad1): track 0.00 -> 18.8 mm, vias 0 -> 2
- net Net-(R7-Pad1): track 0.00 -> 18.1 mm, vias 0 -> 2
- net Earth: track 0.00 -> 15.4 mm
- net Net-(C16-Pad1): track 0.00 -> 12.7 mm
- net /USB & Buttons & LEDs/TX: track 0.00 -> 11.4 mm
- net Net-(R9-Pad1): track 0.00 -> 10.5 mm
- net /USB & Buttons & LEDs/RX: track 0.00 -> 10.4 mm
- net /Thermocouple 1/T-: track 0.00 -> 10.2 mm
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Other:
- rule trace_min: 0.127 -> 0
- board text added: "PWR"
- board text added: "RX"
- board text added: "TX"

Commit message: small bugfixes. Added parts to bom
Parts:
- removed R6, R7: 470R, Resistor_SMD:R_0603_1608Metric
- U8: footprint Package_TO_SOT_THT:TO-92_Inline -> T-962_Upgrade_board:TO-92_Inline
- moved R1 1.46 mm to (138.1, 100.2)
- moved U8 1.46 mm to (134.4, 101.5)
- moved C37 0.64 mm to (134.4, 95.8)
- moved C38 0.64 mm to (132.5, 95.8)
- moved C15 0.30 mm to (148.6, 107.7)
- moved C14 0.30 mm to (150.4, 107.9)
Connections:
- U2 pad 2: Net-(R7-Pad1) -> /USB & Buttons & LEDs/TX
- U2 pad 3: Net-(R6-Pad1) -> /USB & Buttons & LEDs/RX
Routing:
- net Net-(R6-Pad1): track 18.8 -> 0.00 mm, vias 2 -> 0
- net Net-(R7-Pad1): track 18.1 -> 0.00 mm, vias 2 -> 0
- net /USB & Buttons & LEDs/RX: track 10.4 -> 26.4 mm, vias 0 -> 2
- net /USB & Buttons & LEDs/TX: track 11.4 -> 27.1 mm, vias 0 -> 2
- net VDDA: track 87.2 -> 89.4 mm
- net VDD: track 72.7 -> 71.8 mm
- net /SW_IO: track 61.5 -> 62.2 mm
- net VSSA: vias 83 -> 84
- net VSS: vias 98 -> 97
