File: usb.sch (KiCad schematic (older format))
At the start: 20 parts, among them J4 USB_B_Micro, SW1 Boot, SW2 Boot, U2 CH340C

Commit message: Bugfixes in the schematic and started the pcb layout
Connections:
- net VSS: no longer D5.1 (K)
- new net VSSA: D5.1 (K)
Changed lines of the file:
@@
 $Descr A4 11693 8268
 encoding utf-8
-Sheet 3 9
+Sheet 2 9
 Title "USB FTDI & Buttons"
 Date "2020-02-07"
@@
 L power:VSS #PWR?
 U 1 1 5F8E8849
-P 2550 6500
+P 2350 6500
 AR Path="/5DD6D4DA/5DEBB035/5F8E8849" Ref="#PWR?"  Part="1"
 AR Path="/5E15DEC3/5F8E8849" Ref="#PWR?"  Part="1"
@@
 AR Path="/5E1EC3C1/5F8E8849" Ref="#PWR?"  Part="1"
 AR Path="/5E3BDE20/5F8E8849" Ref="#PWR020"  Part="1"
-F 0 "#PWR020" H 2550 6350 50  0001 C CNN
-F 1 "VSS" H 2450 6600 50  0000 C CNN
-F 2 "" H 2550 6500 50  0001 C CNN
-F 3 "" H 2550 6500 50  0001 C CNN
-	1    2550 6500
+F 0 "#PWR020" H 2350 6350 50  0001 C CNN
+F 1 "VSS" H 2350 6650 50  0000 C CNN
+F 2 "" H 2350 6500 50  0001 C CNN
+F 3 "" H 2350 6500 50  0001 C CNN
+	1    2350 6500
 	-1   0    0    1
 $EndComp
@@
 	2350 6300 2350 6500
 Wire Wire Line
-	2350 6500 2550 6500
-Wire Wire Line
-	2550 6500 2700 6500
-Wire Wire Line
 	2700 6500 2700 6300
-Connection ~ 2550 6500
 Wire Notes Line
 	700  4700 3450 4700
@@
 Text Notes 850  4900 0    79   ~ 0
 LED indicators
+$Comp
+L power:VSSA #PWR?
+U 1 1 5F930DE6
+P 2700 6500
+AR Path="/5E3B5CB9/5F930DE6" Ref="#PWR?"  Part="1"
+AR Path="/5F930DE6" Ref="#PWR?"  Part="1"
+AR Path="/5E3D0FD8/5F930DE6" Ref="#PWR?"  Part="1"
+AR Path="/5E3BDE20/5F930DE6" Ref="#PWR0101"  Part="1"
+F 0 "#PWR0101" H 2700 6350 50  0001 C CNN
+F 1 "VSSA" H 2700 6650 50  0000 C CNN
+F 2 "" H 2700 6500 50  0001 C CNN
+F 3 "" H 2700 6500 50  0001 C CNN
+	1    2700 6500
+	-1   0    0    1
+$EndComp
 $EndSCHEMATC

Commit message: small bugfixes. Added parts to bom
Parts:
- removed R6, R7: 470R, Resistor_SMD:R_0603_1608Metric, symbol Device:R
- J4: Link (none) -> https://www.digikey.com/en/products/detail/molex/1050170001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; MPN (none) -> 105017-0001; Manufacturer (none) -> Molex; Package (none) -> SMD/THT; SPN (none) -> WM1399TR-ND; description (none) -> USB - micro B USB 2.0 Receptacle Connector 5 Position Surfa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; lcsc# C136000 -> (none); manf# 105017-0001 -> (none)
- R2, R3, R4, R5: Link (none) -> https://www.digikey.com/en/products/detail/yageo/AC0603JR-0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; MPN (none) -> AC0603JR-0710KL; Manufacturer (none) -> Yageo; Package (none) -> 0603 (1608 Metric); SPN (none) -> 311-10KLECT-ND; description (none) -> 10 ±5% 0.1W, 1/10W Chip Resistor 0603 (1608 Metric) Automot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
- R8, R9: Link (none) -> https://www.digikey.de/product-detail/en/yageo/RC0603JR-074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; MPN (none) -> RC0603JR-07470RL; Manufacturer (none) -> Yageo; Package (none) -> 0603 (1608 Metric); SPN (none) -> 311-470GRCT-ND; description (none) -> 470 Ohms ±5% 0.1W, 1/10W Chip Resistor 0603 (1608 Metric) T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; lcsc# C23179 -> (none); manf# 0603WAF4700T5E -> (none)
- SW1, SW2: Link (none) -> https://www.digikey.com/en/products/detail/e-switch/TL3342F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; MPN (none) -> TL3342F160QG; Manufacturer (none) -> E-Switch; Package (none) -> SMD; SPN (none) -> EG2531TR-ND; description (none) -> Tactile Switch SPST-NO Top Actuated Surface Mount; lcsc# C318889 -> (none); manf# TS-1187A-C-C-B -> (none)
- U2: lcsc# C84681 -> (none); manf# CH340C -> (none)
Connections:
- net RX: now also U2.3 (RXD)
- net TX: now also U2.2 (TXD)

Commit message: Update Readme
Parts:
- added J?: USB_B_Micro, symbol T962upgrade-rescue:USB_B_Micro-Connector
- J4: symbol Connector:USB_B_Micro -> T962upgrade-rescue:USB_B_Micro-Connector
Changed lines of the file:
@@
 	2500 3850 2500 3750
 $Comp
-L Connector:USB_B_Micro J4
+L T962upgrade-rescue:USB_B_Micro-Connector J4
 U 1 1 5E20AD27
 P 2000 2450
@@
 Wire Wire Line
 	5200 2150 5550 2150
+$Comp
+L T962upgrade-rescue:USB_B_Micro-Connector J?
+U 1 1 5FAB3D36
+P -350 2400
+F 0 "J?" H -293 2867 50  0000 C CNN
+F 1 "USB_B_Micro" H -293 2776 50  0000 C CNN
+F 2 "" H -200 2350 50  0001 C CNN
+F 3 "~" H -200 2350 50  0001 C CNN
+	1    -350 2400
+	1    0    0    -1
+$EndComp
 $EndSCHEMATC
